Commit message: Update scaled X5A assets and insert_tube control

File: assets/embodiments/ARX-X5/X5A.urdf (robot description, URDF)
Before this commit: robot X5A, 13 links, 12 joints
Links:
- link x5a_adapter_left_link: geometry collision mesh filename=meshes/XenseWS.STL scale=0.0015 0.0015 0.0015; collision mesh filename=meshes/adapter_left.STL scale=0.0015 0.0015 0.0015
- link x5a_adapter_right_link: geometry collision mesh filename=meshes/XenseWS.STL scale=0.0015 0.0015 0.0015; collision mesh filename=meshes/adapter_right.STL scale=0.0015 0.0015 0.0015
- link x5a_camera: geometry visual mesh filename=meshes/camera.glb scale=1.5 1.5 1.5
- link x5a_camera_base: geometry visual mesh filename=meshes/camera_base.glb scale=1.785123 1.5 1.52975193
- link x5a_link0: geometry collision mesh filename=meshes/x5a_link0.STL scale=1.785123 1.5 1.785123; visual mesh filename=meshes/x5a_link0.STL scale=1.785123 1.5 1.785123
- link x5a_link1: geometry collision mesh filename=meshes/x5a_link1.STL scale=1.785123 1.5 1.785123; visual mesh filename=meshes/x5a_link1.STL scale=1.785123 1.5 1.785123
- link x5a_link2: geometry collision mesh filename=meshes/x5a_link2.STL scale=1.785123 1.5 1.785123; visual mesh filename=meshes/x5a_link2.STL scale=1.785123 1.5 1.785123
- link x5a_link3: geometry collision mesh filename=meshes/x5a_link3.STL scale=1.785123 1.5 1.785123; visual mesh filename=meshes/x5a_link3.STL scale=1.785123 1.5 1.785123
- link x5a_link4: geometry collision mesh filename=meshes/x5a_link4.STL scale=1.785123 1.5 1.785123; visual mesh filename=meshes/x5a_link4.STL scale=1.785123 1.5 1.785123
- link x5a_link5: geometry collision mesh filename=meshes/x5a_link5.STL scale=1.785123 1.5 1.785123; visual mesh filename=meshes/x5a_link5.STL scale=1.785123 1.5 1.785123
- link x5a_link6: geometry collision mesh filename=meshes/x5a_link6.STL scale=1.785123 1.5 1.785123; visual mesh filename=meshes/x5a_link6.STL scale=1.785123 1.5 1.785123
Joints:
- joint x5a_adapter_left_mount: limit lower=0.0 upper=0.025 effort=100 velocity=0.2 -> lower=-0.015 upper=0.06 effort=100 velocity=0.2; origin xyz=0.103025399 0.04999 0.00670962 rpy=0 0 0 -> xyz=0.154538098 0.074985 0.01006443 rpy=0 0 0
- joint x5a_adapter_link_to_xensews_gripper_center: origin xyz=0.18 0.000545 -0.00329038 rpy=3.1415 0 0 -> xyz=0.27 0.0008175 -0.00493557 rpy=3.1415 0 0
- joint x5a_adapter_right_mount: limit lower=0.0 upper=0.025 effort=100 velocity=0.2 -> lower=-0.015 upper=0.06 effort=100 velocity=0.2; origin xyz=0.103025399 -0.0489 0.00670962 rpy=0 0 0 -> xyz=0.154538098 -0.07335 0.01006443 rpy=0 0 0
- joint x5a_camera_joint: origin xyz=-0.032727255 0 0.0595041 rpy=0 0.3491 3.141592653589793 -> xyz=-0.0490908825 0 0.08925615 rpy=0 0.3491 3.141592653589793
- joint x5a_hand_to_camera_mount: origin xyz=0.067834674 0 0 rpy=0 0 -3.1416 -> xyz=0.101752011 0 0 rpy=0 0 -3.1416
- joint x5a_joint1: origin xyz=0 0 0.071999961 rpy=0 0 0 -> xyz=0 0 0.107999942 rpy=0 0 0
- joint x5a_joint2: origin xyz=0.02380164 0 0.04760328 rpy=0 0 0 -> xyz=0.03570246 0 0.07140492 rpy=0 0 0
- joint x5a_joint3: origin xyz=-0.314181648 0 0 rpy=3.1416 0 0 -> xyz=-0.471272472 0 0 rpy=3.1416 0 0
- joint x5a_joint4: origin xyz=0.29157009 0 -0.066644592 rpy=0 0 0 -> xyz=0.437355135 0 -0.099966888 rpy=0 0 0
- joint x5a_joint5: origin xyz=0.080628056 0.0005 -0.102942093 rpy=0 0 0 -> xyz=0.120942084 0.00075 -0.154413139 rpy=0 0 0
- joint x5a_joint6: origin xyz=0.034452874 0 0.102942093 rpy=-3.1416 0 0 -> xyz=0.051679311 0 0.154413139 rpy=-3.1416 0 0
- joint x5a_link6_to_adapter: origin xyz=-0.01 0 0 rpy=0 0 0 -> xyz=-0.015 0 0 rpy=0 0 0

Commit message: fix: update X5A robot configuration

File: assets/embodiments/ARX-X5/X5A.urdf (robot description, URDF)
Before this commit: robot X5A, 13 links, 12 joints
Links:
- link x5a_adapter_left_link: geometry collision mesh filename=meshes/XenseWS.STL scale=0.001 0.001 0.001; collision mesh filename=meshes/adapter_left.STL scale=0.001 0.001 0.001
- link x5a_adapter_right_link: geometry collision mesh filename=meshes/XenseWS.STL scale=0.001 0.001 0.001; collision mesh filename=meshes/adapter_right.STL scale=0.001 0.001 0.001
- link x5a_camera: geometry visual mesh filename=meshes/camera.glb
- link x5a_camera_base: geometry visual mesh filename=meshes/camera_base.glb
- link x5a_link0: geometry collision mesh filename=meshes/base_link.STL; visual mesh filename=meshes/base_link.STL
- link x5a_link1: geometry collision mesh filename=meshes/link1.STL; visual mesh filename=meshes/link1.STL
- link x5a_link2: geometry collision mesh filename=meshes/link2.STL; visual mesh filename=meshes/link2.STL
- link x5a_link3: geometry collision mesh filename=meshes/link3.STL; visual mesh filename=meshes/link3.STL
- link x5a_link4: geometry collision mesh filename=meshes/link4.STL; visual mesh filename=meshes/link4.STL
- link x5a_link5: geometry collision mesh filename=meshes/link5.STL; visual mesh filename=meshes/link5.STL
- link x5a_link6: geometry collision mesh filename=meshes/link6.STL; visual mesh filename=meshes/link6.STL
Joints:
- joint x5a_adapter_left_mount: origin xyz=0.154538098 0.074985 0.01006443 rpy=0 0 0 -> xyz=0.09657 0.04999 0.015638 rpy=0 0 0
- joint x5a_adapter_link_to_xensews_gripper_center: origin xyz=0.27 0.0008175 -0.00493557 rpy=3.1415 0 0 -> xyz=0.151250082 0.000545 -0.002764835 rpy=3.1415 0 0
- joint x5a_adapter_right_mount: origin xyz=0.154538098 -0.07335 0.01006443 rpy=0 0 0 -> xyz=0.09657 -0.0489 0.015638 rpy=0 0 0
- joint x5a_camera_joint: origin xyz=-0.0490908825 0 0.08925615 rpy=0 0.3491 3.141592653589793 -> xyz=-0.0275 0.0 0.05 rpy=0 0.3491 3.141592653589793
- joint x5a_hand_to_camera_mount: origin xyz=0.101752011 0 0 rpy=0 0 -3.1416 -> xyz=0.057 0 0 rpy=0 0 -3.1416
- joint x5a_joint1: origin xyz=0 0 0.107999942 rpy=0 0 0 -> xyz=0 0 0.0605 rpy=0 0 0
- joint x5a_joint2: origin xyz=0.03570246 0 0.07140492 rpy=0 0 0 -> xyz=0.02 0 0.04 rpy=0 0 0
- joint x5a_joint3: origin xyz=-0.471272472 0 0 rpy=3.1416 0 0 -> xyz=-0.264 0 0 rpy=3.1416 0 0
- joint x5a_joint4: origin xyz=0.437355135 0 -0.099966888 rpy=0 0 0 -> xyz=0.245 0 -0.056 rpy=0 0 0
- joint x5a_joint5: origin xyz=0.120942084 0.00075 -0.154413139 rpy=0 0 0 -> xyz=0.06775 0.0005 -0.0865 rpy=0 0 0
- joint x5a_joint6: origin xyz=0.051679311 0 0.154413139 rpy=-3.1416 0 0 -> xyz=0.02895 0 0.0865 rpy=-3.1416 0 0
- joint x5a_link6_to_adapter: origin xyz=-0.015 0 0 rpy=0 0 0 -> xyz=-0.008402782 0 0 rpy=0 0 0
